File: 8BitGen/8BitGen.kicad_pcb (KiCad board)
At the start: 2 copper layers, 0 parts

Commit message: PCB layout
Parts:
- added C1: 0.1u, Capacitor_THT:CP_Radial_Tantal_D5.0mm_P5.00mm, F.Cu at (26.6, 49.8)
- added C2: 10u, Capacitor_THT:CP_Radial_Tantal_D5.0mm_P5.00mm, F.Cu at (139.7, 59.7)
- added C3: 10u, Capacitor_THT:CP_Radial_Tantal_D5.0mm_P5.00mm, F.Cu at (139.7, 52.1)
- added J1: Input Header, Connector_PinHeader_2.54mm:PinHeader_1x07_P2.54mm_Horizontal, F.Cu at (152.4, 39.4)
- added J2: Thru Hole Pads, Connector_PinHeader_2.54mm:PinHeader_1x09_P2.54mm_Vertical, F.Cu at (45.6, 15.8)
- added J3: TRS, Connector_Audio:Jack_3.5mm_CUI_SJ1-3533NG_Horizontal, F.Cu at (63.8, 19.7)
- added U1: 74HC595, Package_DIP:DIP-16_W7.62mm, F.Cu at (49.6, 15.5)
- added U2: SN7404N, Package_DIP:DIP-14_W7.62mm, F.Cu at (70.7, 15.5)
- added U3: LM358, Package_DIP:DIP-8_W7.62mm, F.Cu at (115.6, 35.6)
- added U4: YM3812, Package_DIP:DIP-24_W15.24mm, F.Cu at (26.5, 15.5)
- added U5: YM3014B, Package_DIP:DIP-8_W7.62mm, F.Cu at (143.5, 67.3)
- added X1: SG-531, Oscillator:Oscillator_SeikoEpson_SG-8002DC, F.Cu at (81.5, 17.3)

Commit message: more pcb layout
Parts:
- moved U4 86.9 mm to (104.1, 54.6), turned to 270 degrees
- moved X1 69.1 mm to (115.6, 77.5), turned to 180 degrees
- moved J3 62.3 mm to (125.0, 31.5)
- moved U1 60.4 mm to (69.8, 72.4), turned to 180 degrees
- moved U2 26.8 mm to (80.0, 40.6), turned to 270 degrees
- moved U3 18.1 mm to (127.0, 49.5)
- moved U5 17.3 mm to (127.0, 62.2), turned to 0 degrees
- moved C1 6.76 mm to (33.0, 52.1)
Routing:
- net DO: track 0.00 -> 40.7 mm
- net DAC_CLK: track 0.00 -> 38.3 mm
- net SYNC: track 0.00 -> 35.8 mm
- net D_SOUND: track 0.00 -> 33.9 mm
- net D7: track 0.00 -> 24.3 mm
- net D1: track 0.00 -> 22.2 mm
- net REG_CLK: track 0.00 -> 21.5 mm
- net D6: track 0.00 -> 20.7 mm
- net AUDIO_LINE: track 0.00 -> 18.2 mm
- net D5: track 0.00 -> 17.1 mm
- net DAC_MP: track 0.00 -> 16.3 mm
- net WR_N: track 0.00 -> 14.1 mm
- net D4: track 0.00 -> 13.5 mm
- net BUFF: track 0.00 -> 11.2 mm
- net D3: track 0.00 -> 9.94 mm
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
Commit message: pcb layout
Parts:
- moved C1 107.8 mm to (139.7, 67.6)
- moved J2 70.6 mm to (80.0, 77.5), turned to 90 degrees
- moved J1 66.2 mm to (86.4, 34.8), turned to 90 degrees
- moved X1 37.6 mm to (108.0, 40.6), turned to 0 degrees
- moved J3 0.79 mm to (125.0, 32.3)
Routing:
- net DAC_RB: track 7.18 -> 73.0 mm, vias 0 -> 1
- net AUDIO_LINE: track 18.2 -> 78.7 mm
- net SERIAL_IN: track 0.00 -> 55.6 mm
- net DAC_MP: track 16.3 -> 69.4 mm
- net SERIAL_CLK: track 0.00 -> 51.6 mm
- net REG_CLK: track 21.5 -> 72.5 mm
- net BUFF: track 11.2 -> 59.6 mm
- net 358_CLK: track 3.81 -> 36.6 mm
- net YM_RST_N: track 0.00 -> 27.5 mm
- net WR_N: track 14.1 -> 40.0 mm, vias 0 -> 1
- net YM_A0: track 0.00 -> 19.8 mm
- net D_SOUND: track 33.9 -> 51.0 mm
- net +5V: track 0.00 -> 14.7 mm
- net DAC_CLK: track 38.3 -> 48.5 mm
- net SYNC: track 35.8 -> 44.0 mm
- added copper zone on B.Cu, net +5V
- added copper zone on F.Cu, net GND
Other:
- board outline added: 90.4 x 50.5 mm

Commit message: Add track file
Parts:
- J1: footprint Connector_PinHeader_2.54mm:PinHeader_1x07_P2.54mm_Horizontal -> Connector_PinHeader_2.54mm:PinHeader_1x07_P2.54mm_Vertical
- moved J1 1.14 mm to (86.4, 33.7)
- moved J3 1.12 mm to (125.0, 33.4)
Connections:
- J2 pad 1: AUDIO_LINE -> REG_CLK
- J2 pad 9: REG_CLK -> AUDIO_LINE
Routing:
- net +5V: track 14.7 -> 40.7 mm
- net REG_CLK: track 72.5 -> 51.6 mm
- net AUDIO_LINE: track 78.7 -> 94.9 mm
- net YM_RST_N: track 27.5 -> 28.6 mm
- net YM_A0: track 19.8 -> 21.0 mm
- net WR_N: track 40.0 -> 41.1 mm
- net SERIAL_IN: track 55.6 -> 56.8 mm
- net SERIAL_CLK: track 51.6 -> 52.8 mm
Other:
- board size 90.4 x 50.5 mm -> 88.9 x 47.6 mm
- board text added: "Chiptune Music Board By Liu (Zuguang Liu) Fall 2019"
